File: Project/RetroZ-Main.kicad_pcb (KiCad board)
At the start: 2 copper layers, 100 x 80 mm, 23 parts, among them J1 PJ-102A, J2 Master Bus, SW1 On/Off, SW2 RESET, U1 74HCT04, U2 L7805CV-DG, U3 Z80CPU, U4 max699cpa, Y1 7.3728Mhz

Commit message: finished main board
Parts:
- moved RN2 40.5 mm to (159.8, 73.7)
Routing:
- net ~RESET: track 0.00 -> 125.7 mm, vias 0 -> 7
- net CLK: track 0.00 -> 103.8 mm, vias 0 -> 4
- net /D1: track 0.00 -> 78.6 mm, vias 0 -> 4
- net /D0: track 0.00 -> 77.4 mm, vias 0 -> 2
- net /D2: track 0.00 -> 72.2 mm, vias 0 -> 6
- net /D4: track 0.00 -> 71.1 mm, vias 0 -> 5
- net /D6: track 0.00 -> 68.3 mm, vias 0 -> 4
- net /D3: track 0.00 -> 62.6 mm, vias 0 -> 4
- net /D5: track 0.00 -> 62.1 mm, vias 0 -> 5
- net /D7: track 0.00 -> 56.8 mm, vias 0 -> 4
- net ~WAIT: track 0.00 -> 55.1 mm, vias 0 -> 5
- net ~M1: track 0.00 -> 55.0 mm, vias 0 -> 4
- net ~RD: track 0.00 -> 54.2 mm, vias 0 -> 3
- net /A9: track 0.00 -> 52.7 mm, vias 0 -> 2
- net /A0: track 0.00 -> 49.5 mm, vias 0 -> 2
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- added copper zone on B.Cu, net GND
- added copper zone on F.Cu, net VCC

Commit message: memory board halfway
Parts:
- removed RN2: 2k2, Resistors_THT:R_Array_SIP9
- RN1: value 2k2 -> 10k
- moved J1 20.1 mm to (172.1, 126.4), turned to 180 degrees
- moved C1 12.7 mm to (167.6, 88.3)
- moved C5 12.7 mm to (167.6, 92.7)
- moved C6 12.7 mm to (175.3, 101.0)
- moved C7 12.7 mm to (167.6, 110.5)
- moved SW1 12.7 mm to (182.9, 109.2)
- moved SW2 12.7 mm to (187.3, 80.0)
- moved Y1 12.7 mm to (168.9, 78.7)
- moved C2 12.7 mm to (95.2, 122.6)
- moved J2 12.7 mm to (95.2, 68.6)
- moved REF** 12.7 mm to (90.2, 137.2)
- moved C3 12.7 mm to (120.7, 94.0)
- moved C4 12.7 mm to (149.9, 99.1)
- moved D1 12.7 mm to (186.1, 93.3)
- moved R1 12.7 mm to (156.8, 67.9)
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Routing:
- net VCC: track 0.00 -> 39.2 mm, vias 0 -> 2
- net /D0: track 77.4 -> 44.9 mm, vias 2 -> 1
- net /D1: track 78.6 -> 47.2 mm, vias 4 -> 2
- net /D2: track 72.2 -> 40.9 mm, vias 6 -> 2
- net /D3: track 62.6 -> 41.0 mm, vias 4 -> 2
- net /D7: track 56.8 -> 36.3 mm, vias 4 -> 2
- net /D5: track 62.1 -> 42.8 mm, vias 5 -> 2
- net /D6: track 68.3 -> 49.8 mm, vias 4 -> 2
- net /D4: track 71.1 -> 52.7 mm, vias 5 -> 2
- net ~INT: track 47.1 -> 63.9 mm, vias 5 -> 3
- net Net-(RN1-Pad3): track 28.7 -> 18.5 mm, vias 3 -> 1
- net Net-(RN1-Pad6): track 38.4 -> 44.3 mm
- net ~WAIT: track 55.1 -> 49.9 mm, vias 5 -> 3
- net Net-(D1-Pad2): track 0.00 -> 4.44 mm
- net Net-(R1-Pad1): track 17.6 -> 20.7 mm
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Other:
- board text added: "RetroZ Stack 2018 Main Board Rev. 1 jpgravel@formix.org"
