File: Projects/Main/RetroZ-Main.kicad_pcb (KiCad board)
At the start: 2 copper layers, 100 x 80 mm, 24 parts, among them J1 PJ-102AH, J2 Master Bus, J3 CLOCK SEL, SW1 On/Off, SW2 RESET, U1 74HCT04, U2 L7805CV-DG, U3 Z80CPU, U4 ADM80X, Y1 7.3728Mhz

Commit message: adjusted configuration for JLCPCB plotting
Routing:
- net CLK: track 71.7 -> 69.2 mm, vias 3 -> 1
- net ~RESET: track 122.6 -> 120.8 mm, vias 3 -> 2
