File: Projects/Memory/RetroZ-Memory.kicad_pcb (KiCad board)
At the start: 2 copper layers, 100 x 80 mm, 23 parts, among them J1 Client Bus, U1 74LS32, U10 4002, U2 AT28C64B-15PU, U3 74LS138, U4 74HCT04, U5 74LS08, U6 AS6C4008-55PCN, U7 74HC273, U8 74LS08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

Commit message: simplified schematic
Connections:
- U5 pad 11: /RAM_E -> ~RAM_SEL
- U5 pad 12: ~RAM_SEL -> Net-(U5-Pad12)
- U6 pad 22: /RAM_E -> ~RAM_SEL
- U9 pad 15: ~RAM_SEL -> Net-(U5-Pad12)
Routing:
- net Net-(U5-Pad12): track 0.00 -> 33.6 mm, vias 0 -> 1
- net /RAM_E: track 22.4 -> 0.00 mm, vias 2 -> 0
- net ~RAM_SEL: track 33.6 -> 22.4 mm, vias 1 -> 2
Changed lines of the file:
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@@
   (net 73 DMA1)
   (net 74 DMA2)
-  (net 75 /RAM_E)
+  (net 75 "Net-(U5-Pad12)")
   (net_class Default "This is the default net class."
     (clearance 0.1524)
@@
     (add_net /D6)
     (add_net /D7)
-    (add_net /RAM_E)
     (add_net /~RAMS)
     (add_net A15)
@@
     (add_net "Net-(U3-Pad9)")
     (add_net "Net-(U4-Pad4)")
+    (add_net "Net-(U5-Pad12)")
     (add_net "Net-(U5-Pad6)")
     (add_net "Net-(U5-Pad8)")
@@
       (net 50 "Net-(U4-Pad4)"))
     (pad 11 thru_hole oval (at 7.62 7.62) (size 2.4 1.6) (drill 0.8) (layers *.Cu *.Mask)
-      (net 75 /RAM_E))
+      (net 53 ~RAM_SEL))
     (pad 5 thru_hole oval (at 0 10.16) (size 2.4 1.6) (drill 0.8) (layers *.Cu *.Mask)
       (net 28 CLK))
     (pad 12 thru_hole oval (at 7.62 5.08) (size 2.4 1.6) (drill 0.8) (layers *.Cu *.Mask)
-      (net 53 ~RAM_SEL))
+      (net 75 "Net-(U5-Pad12)"))
     (pad 6 thru_hole oval (at 0 12.7) (size 2.4 1.6) (drill 0.8) (layers *.Cu *.Mask)
       (net 54 "Net-(U5-Pad6)"))
@@
       (net 9 /A6))
     (pad 22 thru_hole oval (at 15.24 25.4) (size 2.4 1.6) (drill 0.8) (layers *.Cu *.Mask)
-      (net 75 /RAM_E))
+      (net 53 ~RAM_SEL))
     (pad 7 thru_hole oval (at 0 15.24) (size 2.4 1.6) (drill 0.8) (layers *.Cu *.Mask)
       (net 8 /A5))
@@
       (net 71 "Net-(U9-Pad7)"))
     (pad 15 thru_hole oval (at 7.62 2.54) (size 2.4 1.6) (drill 0.8) (layers *.Cu *.Mask)
-      (net 53 ~RAM_SEL))
+      (net 75 "Net-(U5-Pad12)"))
     (pad 8 thru_hole oval (at 0 17.78) (size 2.4 1.6) (drill 0.8) (layers *.Cu *.Mask)
       (net 2 GND))
@@
   (segment (start 165.245 103.95) (end 180.485 103.95) (width 0.1524) (layer Top) (net 52))
   (segment (start 182.009 72.454) (end 180.485 70.93) (width 0.1524) (layer Bottom) (net 52))
-  (segment (start 180.467 114.554) (end 179.6415 114.554) (width 0.1524) (layer Bottom) (net 53))
-  (segment (start 179.6415 114.554) (end 178.943 113.8555) (width 0.1524) (layer Bottom) (net 53))
-  (segment (start 178.9425 96.33) (end 165.245 96.33) (width 0.1524) (layer Top) (net 53))
-  (segment (start 178.943 96.3295) (end 178.9425 96.33) (width 0.1524) (layer Top) (net 53))
-  (via (at 178.943 96.3295) (size 0.6858) (drill 0.3302) (layers Top Bottom) (net 53))
-  (segment (start 178.943 113.8555) (end 178.943 96.3295) (width 0.1524) (layer Bottom) (net 53))
-  (segment (start 180.467 114.554) (end 180.467 113.9825) (width 0.1524) (layer Bottom) (net 53))
+  (segment (start 165.245 98.87) (end 161.0355 98.87) (width 0.1524) (layer Top) (net 53))
+  (segment (start 154.3045 93.79) (end 149.37 93.79) (width 0.1524) (layer Top) (net 53))
+  (segment (start 155.3845 92.71) (end 154.3045 93.79) (width 0.1524) (layer Top) (net 53))
+  (segment (start 160.7185 92.71) (end 155.3845 92.71) (width 0.1524) (layer Top) (net 53))
+  (segment (start 160.9725 92.964) (end 160.7185 92.71) (width 0.1524) (layer Top) (net 53))
+  (via (at 160.9725 92.964) (size 0.6858) (drill 0.3302) (layers Top Bottom) (net 53))
+  (segment (start 160.9725 98.933) (end 160.9725 92.964) (width 0.1524) (layer Bottom) (net 53))
+  (via (at 160.9725 98.933) (size 0.6858) (drill 0.3302) (layers Top Bottom) (net 53))
+  (segment (start 161.0355 98.87) (end 160.9725 98.933) (width 0.1524) (layer Top) (net 53))
   (segment (start 180.485 91.25) (end 180.485 105.0295) (width 0.1524) (layer Bottom) (net 54))
   (segment (start 158.26 105.0295) (end 157.625 104.3945) (width 0.1524) (layer Top) (net 54))
@@
   (via (at 184.15 108.7755) (size 0.6858) (drill 0.3302) (layers Top Bottom) (net 74))
   (segment (start 172.847 117.094) (end 172.847 116.459) (width 0.1524) (layer Bottom) (net 74))
-  (segment (start 165.245 98.87) (end 161.0355 98.87) (width 0.1524) (layer Top) (net 75))
-  (segment (start 154.3045 93.79) (end 149.37 93.79) (width 0.1524) (layer Top) (net 75))
-  (segment (start 155.3845 92.71) (end 154.3045 93.79) (width 0.1524) (layer Top) (net 75))
-  (segment (start 160.7185 92.71) (end 155.3845 92.71) (width 0.1524) (layer Top) (net 75))
-  (segment (start 160.9725 92.964) (end 160.7185 92.71) (width 0.1524) (layer Top) (net 75))
-  (via (at 160.9725 92.964) (size 0.6858) (drill 0.3302) (layers Top Bottom) (net 75))
-  (segment (start 160.9725 98.933) (end 160.9725 92.964) (width 0.1524) (layer Bottom) (net 75))
-  (via (at 160.9725 98.933) (size 0.6858) (drill 0.3302) (layers Top Bottom) (net 75))
-  (segment (start 161.0355 98.87) (end 160.9725 98.933) (width 0.1524) (layer Top) (net 75))
+  (segment (start 180.467 114.554) (end 179.6415 114.554) (width 0.1524) (layer Bottom) (net 75))
+  (segment (start 179.6415 114.554) (end 178.943 113.8555) (width 0.1524) (layer Bottom) (net 75))
+  (segment (start 178.9425 96.33) (end 165.245 96.33) (width 0.1524) (layer Top) (net 75))
+  (segment (start 178.943 96.3295) (end 178.9425 96.33) (width 0.1524) (layer Top) (net 75))
+  (via (at 178.943 96.3295) (size 0.6858) (drill 0.3302) (layers Top Bottom) (net 75))
+  (segment (start 178.943 113.8555) (end 178.943 96.3295) (width 0.1524) (layer Bottom) (net 75))
+  (segment (start 180.467 114.554) (end 180.467 113.9825) (width 0.1524) (layer Bottom) (net 75))
   (zone (net 1) (net_name VCC) (layer Top) (hatch edge 0.508)
     (connect_pads (clearance 0.508))

Commit message: adjusted configuration for JLCPCB plotting
Parts:
- added REF***: OSHW-Logo2_14.6x12mm_SilkScreen, Symbols:OSHW-Logo2_14.6x12mm_SilkScreen, F.Cu at (176.5, 101.5)

Commit message: completed Main BOM
Connections:
- U2 pad 27: VCC -> ~MWR
Routing:
- net ~MWR: track 53.7 -> 83.3 mm, vias 1 -> 2
- net VCC: track 20.6 -> 18.1 mm
Changed lines of the file:
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@@
     (links 145)
     (no_connects 0)
-    (area 89.5446 49.4981 190.289701 145.4329)
+    (area 89.5446 49.4981 191.408591 145.4329)
     (thickness 1.6)
     (drawings 1)
-    (tracks 1096)
+    (tracks 1106)
     (zones 0)
     (modules 24)
@@
       (net 24 /D2))
     (pad 27 thru_hole oval (at 15.24 2.54) (size 2.4 1.6) (drill 0.8) (layers *.Cu *.Mask)
-      (net 1 VCC))
+      (net 37 ~MWR))
     (pad 14 thru_hole oval (at 0 33.02) (size 2.4 1.6) (drill 0.8) (layers *.Cu *.Mask)
       (net 2 GND))
@@
   (segment (start 165.245 91.25) (end 168.465 91.25) (width 0.5) (layer F.Cu) (net 1))
   (segment (start 168.465 91.25) (end 168.4655 91.2495) (width 0.5) (layer F.Cu) (net 1))
-  (segment (start 125.24 70.93) (end 125.24 68.39) (width 0.5) (layer B.Cu) (net 1))
   (segment (start 96.774 69.723) (end 96.3845 69.723) (width 0.1524) (layer F.Cu) (net 3))
   (segment (start 96.774 69.723) (end 98.171 69.723) (width 0.1524) (layer F.Cu) (net 3))
@@
   (segment (start 99.695 119.634) (end 99.695 111.4425) (width 0.1524) (layer B.Cu) (net 34))
   (via (at 99.695 119.634) (size 0.6858) (drill 0.3302) (layers F.Cu B.Cu) (net 34))
+  (segment (start 149.37 76.01) (end 144.0175 76.01) (width 0.1524) (layer F.Cu) (net 37))
+  (segment (start 127 71.755) (end 126.175 70.93) (width 0.1524) (layer B.Cu) (net 37))
+  (segment (start 127 76.0095) (end 127 71.755) (width 0.1524) (layer B.Cu) (net 37))
+  (via (at 127 76.0095) (size 0.6858) (drill 0.3302) (layers F.Cu B.Cu) (net 37))
+  (segment (start 132.1435 76.0095) (end 127 76.0095) (width 0.1524) (layer F.Cu) (net 37))
+  (segment (start 133.223 77.089) (end 132.1435 76.0095) (width 0.1524) (layer F.Cu) (net 37))
+  (segment (start 140.5255 77.089) (end 133.223 77.089) (width 0.1524) (layer F.Cu) (net 37))
+  (segment (start 140.7795 76.835) (end 140.5255 77.089) (width 0.1524) (layer F.Cu) (net 37))
+  (segment (start 143.1925 76.835) (end 140.7795 76.835) (width 0.1524) (layer F.Cu) (net 37))
+  (segment (start 144.0175 76.01) (end 143.1925 76.835) (width 0.1524) (layer F.Cu) (net 37))
+  (segment (start 126.175 70.93) (end 125.24 70.93) (width 0.1524) (layer B.Cu) (net 37))
   (segment (start 142.367 119.634) (end 143.3195 119.634) (width 0.1524) (layer F.Cu) (net 37))
   (segment (start 143.3195 119.634) (end 144.78 118.1735) (width 0.1524) (layer F.Cu) (net 37))
