File: Projects/RetroZ-SBC/RetroZ-SBC.kicad_pcb (KiCad board)
At the start: 2 copper layers, 127 x 73.7 mm, 59 parts, among them IC1 PO_RESET, IC2 AT28C256B-15PU, IC3 AS6C62256-55PCN, J1 02x20, J2 01x08, J3 01x08, J4 IEI SELECT, J5 USB_OTG, J6 CLOCK DIV., SW1 RESET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

Commit message: added missing pull-ups and changed git status
Parts:
- removed the U3 at (113.7, 80.6)
- added R13: 10K, Resistors_THT:R_Axial_DIN0207_L6.3mm_D2.5mm_P10.16mm_Horizontal, F.Cu at (95.6, 106.3)
- added R14: 10K, Resistors_THT:R_Axial_DIN0207_L6.3mm_D2.5mm_P10.16mm_Horizontal, F.Cu at (95.6, 103.0)
- J2: value 01x08 -> User Port A; footprint Socket_Strips:Socket_Strip_Straight_1x08_Pitch2.54mm -> Pin_Headers:Pin_Header_Straight_1x08_Pitch2.54mm
- J3: value 01x08 -> User Port B; footprint Socket_Strips:Socket_Strip_Straight_1x08_Pitch2.54mm -> Pin_Headers:Pin_Header_Straight_1x08_Pitch2.54mm
Connections:
- J2 pad 4: Net-(J2-Pad4) -> /INT_0
- J2 pad 5: Net-(J2-Pad5) -> /INT_1
- J2 pad 6: Net-(J2-Pad6) -> /INT_2
- J2 pad 7: Net-(J2-Pad7) -> /INT_3
- J2 pad 8: Net-(J2-Pad8) -> /INT_4
- J3 pad 1: /INT_0 -> Net-(J3-Pad1)
- J3 pad 2: /INT_1 -> Net-(J3-Pad2)
- J3 pad 3: /INT_2 -> Net-(J3-Pad3)
- J3 pad 4: /INT_3 -> Net-(J3-Pad4)
- J3 pad 5: /INT_4 -> Net-(J3-Pad5)
Routing:
- net /~BUSRQ: track 94.2 -> 131.0 mm, vias 5 -> 7
- net /~BUSACK: track 95.3 -> 131.7 mm, vias 3 -> 5
- net /INT_0: track 50.1 -> 78.3 mm, vias 2 -> 4
- net /INT_3: track 33.4 -> 56.3 mm, vias 0 -> 2
- net /INT_4: track 28.6 -> 50.8 mm, vias 0 -> 2
- net /INT_1: track 43.1 -> 64.9 mm
- net /INT_2: track 38.3 -> 60.1 mm
Other:
- board text added: "x 7"
- board text removed: "x 5"
