File: Projects/RetroZ-SBC/RetroZ-SBC.kicad_pcb (KiCad board)
At the start: 2 copper layers, 127 x 73.7 mm, 60 parts, among them IC1 PO_RESET, IC2 AT28C256B-15PU, IC3 AS6C62256-55PCN, J1 02x20, J2 User Port A, J3 User Port B, J4 IEI SELECT, J5 USB_OTG, J6 CLOCK DIV., SW1 RESET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

Commit message: added an url to the board
Other:
- board text added: "http://bit.ly/RetroZ"
Changed lines of the file:
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@@
   (general
     (thickness 1.6)
-    (drawings 160)
+    (drawings 161)
     (tracks 1866)
     (zones 0)
@@
     )
   )
+  (gr_text http://bit.ly/RetroZ (at 100.584 131.8895) (layer F.SilkS)
+    (effects (font (size 1.25 1.25) (thickness 0.2)))
+  )
   (gr_text "x 7" (at 90.678 111.379 90) (layer F.SilkS)
     (effects (font (size 1 1) (thickness 0.15)))
@@
     (effects (font (size 0.75 0.75) (thickness 0.15)))
   )
-  (gr_text "Version 1.0" (at 100.6475 130.6195) (layer F.SilkS)
+  (gr_text "Version 1.0" (at 100.584 129.413) (layer F.SilkS)
     (effects (font (size 1.25 1.25) (thickness 0.2)))
   )
-  (gr_text "RetroZ SBC" (at 100.965 127.635) (layer F.SilkS)
+  (gr_text "RetroZ SBC" (at 100.9015 126.5555) (layer F.SilkS)
     (effects (font (size 3 2.5) (thickness 0.4)))
   )
