File: Projects/RetroZ-disk/RetroZ-disk.sch (KiCad schematic (older format))
At the start: 12 parts

Commit message: Created the schematic
Parts:
- added C1: 0.33uF, Resistors_SMD:R_1206_HandSoldering, symbol Device:C_Small
- added C2: 0.1uF, Resistors_SMD:R_1206_HandSoldering, symbol Device:C_Small
- added C5, C6, C7, C8, C9: 1uF, Resistors_SMD:R_1206_HandSoldering, symbol Device:C_Small
- added R1: 10k, Resistors_SMD:R_1206_HandSoldering, symbol Device:R
- added U4: 7402, symbol 74xx:7402
- C3, C4: renamed from C?; footprint (none) -> Resistors_SMD:R_1206_HandSoldering; Mfr# (none) -> C1206C200K5GACTU
- D1: renamed from D?; value RED LED -> DISK IO; footprint (none) -> LEDs:LED_D5.0mm_Horizontal_O1.27mm_Z3.0mm; Mfr# (none) -> NL-5AR30
- I1: renamed from I?; footprint (none) -> S80:S80-1
- IC1: renamed from IC?; value CD74HC4050M -> CD74HC4050E; footprint SOIC127P600X175-16N -> Housings_DIP:DIP-16_W7.62mm_Socket_LongPads; Description CD74HC4050MG4, Hex Buffer, Converter, HC, Non-Inverting 2 t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 -> Buffers & Line Drivers Hex Non-Inverting; Height 1.75 -> (none); Manufacturer_Part_Number CD74HC4050M -> CD74HC4050E; Mouser Part Number 595-CD74HC4050M -> 595-CD74HC4050E; Mouser Price/Stock https://www.mouser.com/Search/Refine.aspx?Keyword=595-CD74H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 -> https://www.mouser.ca/ProductDetail/Texas-Instruments/CD74H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; RS Part Number 0527760 -> (none); RS Price/Stock http://uk.rs-online.com/web/p/products/0527760 -> (none)
- J1: renamed from J?; footprint (none) -> Connectors_Card:MicroSd_Wurth_693072010801; Mfr# (none) -> 693072010801; Mouser (none) -> https://www.mouser.ca/productdetail/wurth-electronics/69307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
- J2: renamed from J?; footprint (none) -> Pin_Headers:Pin_Header_Straight_2x08_Pitch2.54mm; Mfr# (none) -> 87914-1616
- R2: renamed from R?; footprint (none) -> Resistors_SMD:R_1206_HandSoldering; Mfr# (none) -> CRCW1206150RFKEAC
- U1: renamed from U?; footprint (none) -> TO_SOT_Packages_SMD:SOT-223-3_TabPin2; Field4 (none) -> UA78M33CDCYR
- U2: renamed from U?; footprint (none) -> Housings_DIP:DIP-16_W7.62mm_Socket_LongPads; Mfr# (none) -> SN74HC138N
- U3: renamed from U?; footprint DIL28 -> Housings_DIP:DIP-28_W7.62mm_Socket_LongPads
- Y1: renamed from Y?; footprint (none) -> Crystals:Crystal_HC49-4H_Vertical; Mft# (none) -> 9B-20.000MAAJ-B; Package (none) -> HC-49/S
Connections:
- net GND: now also C1.2, C2.2, C5.2, C6.2, C7.2, C8.2, C9.2
- net MISO: now also IC1.4 (2Y); no longer IC1.5 (2A)
- net VCC: now also C1.1, C7.1, C8.1, C9.1, R1.2; no longer U3.21 (AREF)
- net VDD: now also C2.1, C5.1, C6.1
- net ~IORQ: now also U4.2; no longer U3.28 ((PCINT13/SCL/ADC5)PC5)
- net ~SEL: now also U4.3; no longer U3.27 ((PCINT12/SDA/ADC4)PC4)
- net ~WAIT: now reaches I1.33 (~WAIT~)
- net ~WAIT: now also U3.28 ((PCINT13/SCL/ADC5)PC5)
- net at J1.7 (DAT0): now also IC1.5 (2A); no longer IC1.4 (2Y)
- new net: R1.1, U3.21 (AREF)
- new net: U4.1, U4.5, U4.6
- new net ~CS: U3.27 ((PCINT12/SDA/ADC4)PC4), U4.4
- no-connect marks 40 -> 42
Other:
- note added: "5V to 3.3V,500mA"
- note added: "Decoupling capacitors"
- note added: "IO Base Address: 0b001SSSMM\nWhere SSS the IO SEL bits and\nMM are the IO Mode bits"
- moved on the sheet: C3, C4, D1, I1, IC1, J1, J2, R2, U1, U2, U3, Y1
